File: hardware/cpld.brd (EAGLE design)
At the start: 72.7 x 67.9 mm, 31 parts, among them IC2 LM1117IMPX-3.3

Commit message: Board updated
Parts:
- added C12: (no value), rcl:C0402
- added R8: (no value), rcl:R0603
- added S1: DTSM-3, switch-tact:DTSM-3
- moved JP3 3.00 mm to (8.28, 42.7), flipped to the bottom
- moved C7 1.72 mm to (38.7, 19.8)
- moved C1 0.43 mm to (22.5, 30.6)
Connections:
- new net GSR: R8.2, S1.1, U$2.99
- new net IO21: JP3.17, U$2.76
- new net IO22: JP3.18, U$2.77
- new net IO23: JP3.15, U$2.78
- new net IO24: JP3.16, U$2.79
- new net IO25: JP3.13, U$2.80
- new net IO26: JP3.14, U$2.81
- new net IO27: JP3.11, U$2.82
- new net IO28: JP3.12, U$2.85
- new net IO29: JP3.9, U$2.86
- new net IO30: JP3.10, U$2.87
- new net IO31: JP3.7, U$2.89
- new net IO32: JP3.8, U$2.90
- new net IO33: JP3.5, U$2.91
- new net IO34: JP3.6, U$2.92
- new net IO35: JP3.3, U$2.93
- new net IO36: JP3.4, U$2.94
- new net IO37: U$2.95
- net 3V: now also C12.1, R8.1
- net CLK: now also U$2.23; no longer U$2.24
- net D2A: now also U$2.24; no longer U$2.23
- net GND: now also C12.2, JP3.1, JP3.2, S1.2
Routing:
- net IO21: track 0.00 -> 22.3 mm
- net IO23: track 0.00 -> 21.7 mm
- net IO25: track 0.00 -> 21.0 mm
- net IO27: track 0.00 -> 20.4 mm
- net IO29: track 0.00 -> 20.2 mm
- net IO31: track 0.00 -> 19.7 mm
- net IO33: track 0.00 -> 19.1 mm
- net IO22: track 0.00 -> 18.9 mm
- net IO35: track 0.00 -> 18.5 mm
- net IO24: track 0.00 -> 18.3 mm
- net IO26: track 0.00 -> 17.7 mm
- net IO28: track 0.00 -> 17.4 mm
- net IO30: track 0.00 -> 16.8 mm
- net IO32: track 0.00 -> 16.4 mm
- net IO34: track 0.00 -> 15.7 mm
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
Commit message: Boards updated
Changed lines of the file:
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@@
 <contactref element="R2" pad="1"/>
 <contactref element="SV1" pad="4"/>
-<wire x1="64.08" y1="41.33" x2="64.77" y2="40.64" width="0.2667" layer="1"/>
-<wire x1="64.77" y1="40.64" x2="67.31" y2="40.64" width="0.2667" layer="1"/>
-<wire x1="67.31" y1="40.64" x2="67.945" y2="41.275" width="0.2667" layer="1"/>
 <wire x1="67.945" y1="41.275" x2="67.945" y2="43.1" width="0.2667" layer="1"/>
 <wire x1="67.945" y1="43.1" x2="66.675" y2="44.37" width="0.2667" layer="1"/>
 <wire x1="65.3184" y1="44.37" x2="66.675" y2="44.37" width="0.4064" layer="1"/>
+<wire x1="64.8462" y1="40.5638" x2="67.2338" y2="40.5638" width="0.2667" layer="1"/>
+<wire x1="67.2338" y1="40.5638" x2="67.945" y2="41.275" width="0.2667" layer="1"/>
+<wire x1="64.8462" y1="40.5638" x2="64.08" y2="41.33" width="0.2667" layer="1"/>
 </signal>
 <signal name="TDI">

Commit message: Hardware project updates and fixes
Parts:
- removed JP3: (no value), pinhead:2X10
- added JP5: (no value), pinhead:2X09
- added R9: (no value), rcl:R0603
- C11, C12, C2: device rcl:C0402 -> rcl:C0603
- C15: value (none) -> 22uF
- C30: value (none) -> 22 uF
- C8, C9: value (none) -> 1 uF
- R3: value (none) -> 0R
- moved C12 2.54 mm to (17.1, 38.1)
- moved C11 1.60 mm to (37.7, 50.8), turned to 45 degrees
- moved C2 0.43 mm to (40.1, 27.4)
- moved C3 0.10 mm to (35.9, 20.9)
Connections:
- net 3V: now also R9.1
- net DCF: now also R9.2
- net GND: now also JP5.17, JP5.18; no longer JP3.1, JP3.2, U$3.1
- net IO21: now also JP5.15; no longer JP3.17
- net IO22: now also JP5.16; no longer JP3.18
- net IO23: now also JP5.13; no longer JP3.15
- net IO24: now also JP5.14; no longer JP3.16
- net IO25: now also JP5.11; no longer JP3.13
- net IO26: now also JP5.12; no longer JP3.14
- net IO27: now also JP5.9; no longer JP3.11
- net IO28: now also JP5.10; no longer JP3.12
- net IO29: now also JP5.7; no longer JP3.9
- net IO30: now also JP5.8; no longer JP3.10
- net IO31: now also JP5.5; no longer JP3.7
- net IO32: now also JP5.6; no longer JP3.8
- net IO33: now also JP5.3; no longer JP3.5
- net IO34: now also JP5.4; no longer JP3.6
- net IO35: now also JP5.1; no longer JP3.3
- net IO36: now also JP5.2; no longer JP3.4
Routing:
- net N$1: track 23.6 -> 18.5 mm
- net 3V: track 198.8 -> 202.0 mm
- net 1V8: track 39.1 -> 36.1 mm
- net IO35: track 18.5 -> 15.9 mm
- net IO30: track 16.8 -> 14.3 mm
- net IO29: track 20.2 -> 17.6 mm
- net IO23: track 21.7 -> 19.1 mm
- net IO22: track 18.9 -> 16.4 mm
- net IO34: track 15.7 -> 13.2 mm
- net IO32: track 16.4 -> 13.8 mm
- net IO24: track 18.3 -> 15.8 mm
- net IO36: track 15.1 -> 12.5 mm
- net IO31: track 19.7 -> 17.2 mm
- net IO28: track 17.4 -> 14.9 mm
- net IO27: track 20.4 -> 17.9 mm
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