File: hardware/cpld.sch (EAGLE design)
At the start: 31 parts, among them IC2 LM1117IMPX-3.3

Commit message: Board updated
Parts:
- added C12: (no value), rcl:C-EUC0402
- added R8: (no value), rcl:R-EU_R0603
- added S1: DTSM-3, switch-tact:DTSM-3
Connections:
- new net GSR: R8.2, S1.1, U$2.IO80
- new net IO21: JP3.17, U$2.IO61
- new net IO22: JP3.18, U$2.IO62
- new net IO23: JP3.15, U$2.IO63
- new net IO24: JP3.16, U$2.IO64
- new net IO25: JP3.13, U$2.IO65
- new net IO26: JP3.14, U$2.IO66
- new net IO27: JP3.11, U$2.IO67
- new net IO28: JP3.12, U$2.IO68
- new net IO29: JP3.9, U$2.IO69
- new net IO30: JP3.10, U$2.IO70
- new net IO31: JP3.7, U$2.IO71
- new net IO32: JP3.8, U$2.IO72
- new net IO33: JP3.5, U$2.IO73
- new net IO34: JP3.6, U$2.IO74
- new net IO35: JP3.3, U$2.IO75
- new net IO36: JP3.4, U$2.IO76
- new net IO37: U$2.IO77
- net 3V: now also C12.1, R8.1
- net CLK: now also U$2.IO20; no longer U$2.IO21
- net D2A: now also U$2.IO21; no longer U$2.IO20
- net GND: now also C12.2, JP3.1, JP3.2, S1.2
Other:
- moved on the sheet: C11, C2, C8, C9

Commit message: Hardware project updates and fixes
Parts:
- removed JP3: (no value), pinhead:PINHD-2X10
- added JP5: (no value), pinhead:PINHD-2X9
- added R9: (no value), rcl:R-EU_R0603
- C11, C12, C2: device rcl:C-EUC0402 -> rcl:C-EUC0603
- C15: value (none) -> 22uF
- C30: value (none) -> 22 uF
- C8, C9: value (none) -> 1 uF
- R3: value (none) -> 0R
Connections:
- net 3V: now also R9.1
- net DCF: now also R9.2
- net GND: now also JP5.17, JP5.18; no longer JP3.1, JP3.2, U$3.TRI
- net IO21: now also JP5.15; no longer JP3.17
- net IO22: now also JP5.16; no longer JP3.18
- net IO23: now also JP5.13; no longer JP3.15
- net IO24: now also JP5.14; no longer JP3.16
- net IO25: now also JP5.11; no longer JP3.13
- net IO26: now also JP5.12; no longer JP3.14
- net IO27: now also JP5.9; no longer JP3.11
- net IO28: now also JP5.10; no longer JP3.12
- net IO29: now also JP5.7; no longer JP3.9
- net IO30: now also JP5.8; no longer JP3.10
- net IO31: now also JP5.5; no longer JP3.7
- net IO32: now also JP5.6; no longer JP3.8
- net IO33: now also JP5.3; no longer JP3.5
- net IO34: now also JP5.4; no longer JP3.6
- net IO35: now also JP5.1; no longer JP3.3
- net IO36: now also JP5.2; no longer JP3.4
