File: hardware/display.brd (EAGLE design)
At the start: 216.8 x 99.9 mm, 41 parts

Commit message: Boards updated
Parts:
- added C1, C2: (no value), rcl:SMC_D
- added C13, C14: (no value), rcl:C0603
- added C15: (no value), rcl:SMC_B
- added C30: (no value), rcl:SMC_C
- added F3: SMF_OMNIBLOK_154.062, _hhn_littlefuse_Nano2SMF_2:NANO2_SMF_FUSEBLOCK
- added IC5: 7805DT, linear:TO252
- added Q4: (no value), transistor-power:SO-08
- added R33: 1k, rcl:R0603
- added S1, S2, S3, S4: (no value), switch-omron:B3F-40XX
- moved R25 32.2 mm to (180.8, 91.4)
- moved R29 32.2 mm to (180.8, 38.1)
- moved R19 32.2 mm to (137.7, 91.4)
- moved DIS1 32.2 mm to (60.3, 29.8)
- moved DIS2 32.2 mm to (156.8, 29.8)
- moved DIS3 32.2 mm to (108.6, 29.8)
- moved DIS5 32.2 mm to (12.1, 29.8)
- moved JP2 32.2 mm to (85.7, 6.67)
- moved R1 32.2 mm to (38.6, 91.4)
- moved R10 32.2 mm to (89.4, 91.4)
- moved R11 32.2 mm to (86.9, 38.1)
- moved R12 32.2 mm to (84.3, 38.1)
- moved R13 32.2 mm to (81.8, 38.1)
- moved R14 32.2 mm to (81.8, 91.4)
- moved R15 32.2 mm to (79.2, 91.4)
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Connections:
- new net KEY_1: JP2.2, S1.1, S1.2
- new net KEY_2: JP2.1, S2.1, S2.2
- new net KEY_3: JP2.39, S3.1, S3.2
- new net KEY_4: JP2.40, S4.1, S4.2
- new net N$3: F3.2
- new net N$4: Q4.4, R33.2
- new net N$52: F3.1, Q4.5, Q4.6, Q4.7, Q4.8
- net 5V: now also C14.1, C15.+, IC5.2
- net 9V: now also C1.+, C13.1, C2.+, C30.+, IC5.1, Q4.1, Q4.2, Q4.3
- net GND: now also C1.-, C13.2, C14.2, C15.-, C2.-, C30.-, IC5.3, R33.1, S1.3, S1.4, S2.3, S2.4, S3.3, S3.4, S4.3, S4.4
Routing:
- net 5V: track 5.08 -> 81.6 mm
- net KEY_4: track 0.00 -> 75.3 mm
- net KEY_1: track 0.00 -> 75.0 mm
- net KEY_3: track 0.00 -> 37.6 mm
- net KEY_2: track 0.00 -> 37.6 mm
- net 9V: track 180.6 -> 201.7 mm
- net N$4: track 0.00 -> 1.69 mm
- added copper zone on layer 16, net N$3
- added copper zone on layer 16, net N$52

Commit message: Hardware project updates and fixes
Parts:
- R1, R2, R3, R4, R5, R6, R7: value (none) -> 220R
- R8: value (none) -> 470R
Changed lines of the file:
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@@
 <element name="DIS2" library="display-kingbright" package="SX23-XX" value="SA23-11" x="156.845" y="29.845"/>
 <element name="DIS3" library="display-kingbright" package="SX23-XX" value="SA23-11" x="108.585" y="29.845"/>
-<element name="R1" library="rcl" package="R0603" value="" x="38.608" y="91.44" rot="MR90"/>
-<element name="R2" library="rcl" package="R0603" value="" x="41.148" y="91.44" rot="MR90"/>
-<element name="R3" library="rcl" package="R0603" value="" x="38.608" y="38.1" rot="MR270"/>
-<element name="R4" library="rcl" package="R0603" value="" x="36.068" y="38.1" rot="MR270"/>
-<element name="R5" library="rcl" package="R0603" value="" x="33.528" y="38.1" rot="MR270"/>
-<element name="R6" library="rcl" package="R0603" value="" x="33.528" y="91.44" rot="MR90"/>
-<element name="R7" library="rcl" package="R0603" value="" x="30.988" y="91.44" rot="MR90"/>
-<element name="R8" library="rcl" package="R0603" value="" x="36.068" y="91.44" rot="MR90"/>
+<element name="R1" library="rcl" package="R0603" value="220R" x="38.608" y="91.44" rot="MR90"/>
+<element name="R2" library="rcl" package="R0603" value="220R" x="41.148" y="91.44" rot="MR90"/>
+<element name="R3" library="rcl" package="R0603" value="220R" x="38.608" y="38.1" rot="MR270"/>
+<element name="R4" library="rcl" package="R0603" value="220R" x="36.068" y="38.1" rot="MR270"/>
+<element name="R5" library="rcl" package="R0603" value="220R" x="33.528" y="38.1" rot="MR270"/>
+<element name="R6" library="rcl" package="R0603" value="220R" x="33.528" y="91.44" rot="MR90"/>
+<element name="R7" library="rcl" package="R0603" value="220R" x="30.988" y="91.44" rot="MR90"/>
+<element name="R8" library="rcl" package="R0603" value="470R" x="36.068" y="91.44" rot="MR90"/>
 <element name="R9" library="rcl" package="R0603" value="" x="86.868" y="91.44" rot="MR90"/>
 <element name="R10" library="rcl" package="R0603" value="" x="89.408" y="91.44" rot="MR90"/>
