File: hardware/display.sch (EAGLE design)
At the start: 41 parts

Commit message: Boards updated
Parts:
- added C1, C2: (no value), rcl:CPOL-EUSMCD
- added C13, C14: (no value), rcl:C-EUC0603
- added C15: (no value), rcl:CPOL-EUSMCB
- added C30: (no value), rcl:CPOL-EUSMCC
- added F3: SMF_OMNIBLOK_154.062, _hhn_littlefuse_Nano2SMF_2:SMF_OMNIBLOK_154.062
- added IC5: 7805DT, linear:7805DT
- added Q4: (no value), transistor-power:P-MOSFET-SO8
- added R33: 1k, rcl:R-EU_R0603
- added S1, S2, S3, S4: (no value), switch-omron:40-XX
Connections:
- new net KEY_1: JP2.2, S1.S, S1.S1
- new net KEY_2: JP2.1, S2.S, S2.S1
- new net KEY_3: JP2.39, S3.S, S3.S1
- new net KEY_4: JP2.40, S4.S, S4.S1
- new net N$3: F3.2
- new net N$4: Q4.G, R33.2
- new net N$52: F3.1, Q4.D
- net 5V: now also C14.1, C15.+, IC5.VO
- net 9V: now also C1.+, C13.1, C2.+, C30.+, IC5.VI, Q4.S
- net GND: now also C1.-, C13.2, C14.2, C15.-, C2.-, C30.-, IC5.GND, R33.1, S1.P, S1.P1, S2.P, S2.P1, S3.P, S3.P1, S4.P, S4.P1

Commit message: Hardware project updates and fixes
Parts:
- R1, R2, R3, R4, R5, R6, R7: value (none) -> 220R
- R8: value (none) -> 470R
Changed lines of the file:
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@@
 <part name="DIS2" library="display-kingbright" deviceset="SA23-11" device=""/>
 <part name="DIS3" library="display-kingbright" deviceset="SA23-11" device=""/>
-<part name="R1" library="rcl" deviceset="R-EU_" device="R0603"/>
-<part name="R2" library="rcl" deviceset="R-EU_" device="R0603"/>
-<part name="R3" library="rcl" deviceset="R-EU_" device="R0603"/>
-<part name="R4" library="rcl" deviceset="R-EU_" device="R0603"/>
-<part name="R5" library="rcl" deviceset="R-EU_" device="R0603"/>
-<part name="R6" library="rcl" deviceset="R-EU_" device="R0603"/>
-<part name="R7" library="rcl" deviceset="R-EU_" device="R0603"/>
-<part name="R8" library="rcl" deviceset="R-EU_" device="R0603"/>
+<part name="R1" library="rcl" deviceset="R-EU_" device="R0603" value="220R"/>
+<part name="R2" library="rcl" deviceset="R-EU_" device="R0603" value="220R"/>
+<part name="R3" library="rcl" deviceset="R-EU_" device="R0603" value="220R"/>
+<part name="R4" library="rcl" deviceset="R-EU_" device="R0603" value="220R"/>
+<part name="R5" library="rcl" deviceset="R-EU_" device="R0603" value="220R"/>
+<part name="R6" library="rcl" deviceset="R-EU_" device="R0603" value="220R"/>
+<part name="R7" library="rcl" deviceset="R-EU_" device="R0603" value="220R"/>
+<part name="R8" library="rcl" deviceset="R-EU_" device="R0603" value="470R"/>
 <part name="R9" library="rcl" deviceset="R-EU_" device="R0603"/>
 <part name="R10" library="rcl" deviceset="R-EU_" device="R0603"/>
